File: hardware/Make files/Active/CAN_Firewall.kicad_pcb (KiCad board)
At the start: 2 copper layers, 68 x 58 mm, 80 parts, among them CON1 BARREL_JACK, CON2 AVR-JTAG-10, CON3 AVR-AW-6, J1 +5V_SRC, J2 DB9, J3 DB9, P1 USB_OTG, P2 USB_OTG, P3 DIAG Port, SW1 SPST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

Commit message: Optimization of: route, silk, 3d
Parts:
- C7: footprint Capacitors_Tantalum_SMD:TantalC_SizeA_EIA-3216_Reflow -> Capacitors_SMD:c_elec_6.3x5.3
- CON1: footprint Custom Parts:RAPC722X -> Connect:BARREL_JACK
- CON2: footprint Socket_Strips:Socket_Strip_Straight_2x05 -> Pin_Headers:Pin_Header_Straight_2x05; moved to F.Cu
- CON3: footprint Socket_Strips:Socket_Strip_Straight_2x03 -> Pin_Headers:Pin_Header_Straight_2x03; moved to F.Cu
- D3: footprint Diodes_SMD:SMB_Standard -> Diodes_SMD:SMB_Handsoldering
- J1: footprint Socket_Strips:Socket_Strip_Straight_1x03 -> Pin_Headers:Pin_Header_Straight_1x03
- P3: footprint Socket_Strips:Socket_Strip_Straight_1x12 -> Pin_Headers:Pin_Header_Straight_1x12
- moved D3 25.4 mm to (75.4, 116.5), turned to 90 degrees
- moved C1 17.1 mm to (43.9, 130.0)
- moved R15 7.50 mm to (75.5, 110.0)
- moved C11 7.02 mm to (60.0, 129.5), turned to 0 degrees
- moved CON1 7.02 mm to (85.0, 112.0), turned to 270 degrees
- moved C8 5.21 mm to (47.8, 123.7)
- moved C6 4.50 mm to (48.5, 130.0)
- moved R20 4.50 mm to (53.0, 130.0)
- moved C7 1.45 mm to (50.5, 118.2), turned to 270 degrees
- moved D6 1.20 mm to (75.5, 107.5)
- turned CON2 to 90 degrees
- turned CON3 to 90 degrees
- turned J1 to 270 degrees
- turned P3 to 270 degrees
Routing:
- net GND: track 385.2 -> 418.1 mm, vias 67 -> 69
- net IVI_INT: track 30.7 -> 39.4 mm
- net Net-(D6-Pad2): track 9.57 -> 3.27 mm
- net Net-(R20-Pad1): track 5.65 -> 10.6 mm
- net IVI_CANH: track 27.1 -> 31.3 mm
- net Net-(C1-Pad1): track 15.1 -> 19.1 mm
- net +12V: track 105.5 -> 101.7 mm, vias 4 -> 5
- net Net-(C2-Pad1): track 0.00 -> 2.41 mm
- net CAR_CANH: track 32.7 -> 34.3 mm
- net +5V: track 182.2 -> 183.2 mm
- net LOOP_A: track 37.4 -> 38.4 mm
- net CAR_CANL: track 37.7 -> 38.6 mm
- net IVI_STBY: track 33.1 -> 32.5 mm
- net LOOP_B: track 35.7 -> 35.2 mm
Other:
- board text added: "Jaguar Land Rover CANBUS Firewall V1.2 Open Source Hardware Jesse Banks 2016"
- board text added: "Power"
- board text removed: "Jaguar Land Rovver CANBUS Firewall V1.11 Open Source Hardware Jesse Banks 2015"
- board text removed: "Power "ON" LED"

Commit message: Minor chages
Parts:
- moved C8 1.24 mm to (49.0, 124.0)
- moved C7 0.70 mm to (50.5, 117.5)
- moved FB1 0.50 mm to (49.0, 127.0)
Routing:
- net VBUS: track 21.4 -> 22.7 mm
- net +12V: track 101.7 -> 100.7 mm
Changed lines of the file:
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@@
   (general
     (links 223)
-    (no_connects 0)
+    (no_connects 52)
     (area 39.949999 104.949999 108.050001 163.050001)
     (thickness 1.6)
     (drawings 70)
-    (tracks 1447)
+    (tracks 1448)
     (zones 0)
     (modules 80)
@@
   )
   (module "Custom Parts:R_0603_sm" (layer F.Cu)
-    (at 47.8 123.7 180)
+    (at 49 124 180)
     (descr "Resistor SMD 0603, reflow soldering, Vishay (see dcrcw.pdf)")
     (tags "resistor 0603")
@@
   )
   (module "Custom Parts:Diode_0805_12_SM" (layer F.Cu)
-    (at 49.5 127 180)
+    (at 49 127 180)
     (descr "Resistor SMD 0805, reflow soldering, Vishay (see dcrcw.pdf)")
     (tags "resistor 0805")
@@
   )
   (module Capacitors_SMD:c_elec_6.3x5.3 (layer F.Cu)
-    (at 50.5 118.2 270)
+    (at 50.5 117.5 270)
     (descr "SMT capacitor, aluminium electrolytic, 6.3x5.3")
     (attr smd)
@@
   (segment (start 99.7 123.3) (end 102.8 123.3) (width 0.25) (layer F.Cu) (net 4))
   (segment (start 99.425 123.025) (end 99.7 123.3) (width 0.25) (layer F.Cu) (net 4))
-  (segment (start 47.6 127.5) (end 47.6 129.3) (width 0.5) (layer B.Cu) (net 5))
+  (segment (start 48.3 130) (end 48.3 129.2) (width 0.5) (layer B.Cu) (net 5))
+  (segment (start 48.3 129.2) (end 52 125.5) (width 0.5) (layer B.Cu) (net 5))
+  (via (at 52 125.5) (size 0.75) (drill 0.5) (layers F.Cu B.Cu) (net 5))
+  (segment (start 42.6 128.6) (end 46.9 128.6) (width 0.5) (layer B.Cu) (net 5))
+  (segment (start 46.9 128.6) (end 48.3 130) (width 0.5) (layer B.Cu) (net 5))
   (segment (start 48.3 130) (end 47.6 130) (width 0.5) (layer F.Cu) (net 5))
   (via (at 48.3 130) (size 0.75) (drill 0.5) (layers F.Cu B.Cu) (net 5))
   (segment (start 47.6 129.3) (end 48.3 130) (width 0.5) (layer B.Cu) (net 5))
   (segment (start 42.6 128.6) (end 42.6 128.5) (width 0.5) (layer B.Cu) (net 5))
-  (segment (start 42.6 128.5) (end 43.6 127.5) (width 0.5) (layer B.Cu) (net 5))
   (segment (start 42.54 138.809) (end 42.54 128.66) (width 0.5) (layer B.Cu) (net 5))
   (segment (start 42.55 128.55) (end 42.55 126.5) (width 0.5) (layer F.Cu) (net 5))
@@
   (segment (start 94.1 123.9) (end 96.6 123.9) (width 0.5) (layer B.Cu) (net 5))
   (via (at 94.1 123.9) (size 0.75) (drill 0.5) (layers F.Cu B.Cu) (net 5))
-  (via (at 48.5 125.6) (size 0.75) (drill 0.5) (layers F.Cu B.Cu) (net 5))
-  (segment (start 52.1 125.6) (end 48.5 125.6) (width 0.5) (layer F.Cu) (net 5))
   (segment (start 52.75 124.95) (end 52.1 125.6) (width 0.5) (layer F.Cu) (net 5))
-  (segment (start 48.5 127) (end 48.5 125.6) (width 0.5) (layer B.Cu) (net 5))
-  (segment (start 48.5 127) (end 48 127.5) (width 0.5) (layer B.Cu) (net 5))
-  (segment (start 48 127.5) (end 47.6 127.5) (width 0.5) (layer B.Cu) (net 5))
-  (segment (start 47.6 127.5) (end 43.6 127.5) (width 0.5) (layer B.Cu) (net 5))
   (segment (start 53 124.7) (end 52.75 124.95) (width 0.5) (layer F.Cu) (net 5))
   (segment (start 105 128.5) (end 103.9 128.5) (width 0.5) (layer F.Cu) (net 5))
@@
   (segment (start 62.2 142.2) (end 62.2 142.6) (width 0.25) (layer F.Cu) (net 16))
   (segment (start 64.15 140.25) (end 62.2 142.2) (width 0.25) (layer F.Cu) (net 16))
+  (segment (start 44.750002 128.1) (end 46.783947 128.1) (width 0.25) (layer F.Cu) (net 18))
+  (segment (start 46.783947 128.1) (end 47.25 128.1) (width 0.25) (layer F.Cu) (net 18))
+  (segment (start 47.25 128.1) (end 48.05 127.3) (width 0.25) (layer F.Cu) (net 18))
+  (segment (start 48.05 127.3) (end 48.05 127) (width 0.25) (layer F.Cu) (net 18))
   (segment (start 44.6 126.6) (end 44.6 127.949998) (width 0.25) (layer F.Cu) (net 18))
   (segment (start 44.6 123.35) (end 44.6 126.6) (width 0.25) (layer F.Cu) (net 18))
   (segment (start 45.45 122.5) (end 44.6 123.35) (width 0.25) (layer F.Cu) (net 18))
-  (segment (start 47.45 128.1) (end 48.55 127) (width 0.25) (layer F.Cu) (net 18))
-  (segment (start 44.750002 128.1) (end 47.45 128.1) (width 0.25) (layer F.Cu) (net 18))
   (segment (start 44.6 127.949998) (end 44.750002 128.1) (width 0.25) (layer F.Cu) (net 18))
   (segment (start 45.45 122.5) (end 45.45 121.55) (width 0.25) (layer F.Cu) (net 18))
-  (segment (start 48.55 127) (end 48.55 127.15) (width 0.5) (layer F.Cu) (net 18))
   (segment (start 83.95 128.5) (end 83.95 128.45) (width 0.25) (layer F.Cu) (net 19))
   (segment (start 83.95 128.45) (end 85.4 127) (width 0.25) (layer F.Cu) (net 19))
@@
   (segment (start 76.4 110) (end 76.4 109.35) (width 0.25) (layer F.Cu) (net 28))
   (segment (start 76.4 109.35) (end 74.55 107.5) (width 0.25) (layer F.Cu) (net 28))
+  (segment (start 54.42 126.5) (end 54.42 126.6524) (width 0.25) (layer F.Cu) (net 29))
+  (segment (start 54.42 126.6524) (end 54.0724 127) (width 0.25) (layer F.Cu) (net 29))
+  (segment (start 54.0724 127) (end 50.55 127) (width 0.25) (layer F.Cu) (net 29))
+  (segment (start 50.55 127) (end 49.95 127) (width 0.25) (layer F.Cu) (net 29))
   (segment (start 63 134) (end 61.6 134) (width 0.25) (layer B.Cu) (net 29))
   (segment (start 58.7 131.1) (end 61.6 134) (width 0.25) (layer B.Cu) (net 29))
@@
   (via (at 63.1 134.1) (size 0.6) (drill 0.4) (layers F.Cu B.Cu) (net 29))
   (segment (start 64.8 137.299998) (end 64.8 137.25) (width 0.25) (layer F.Cu) (net 29))
-  (segment (start 50.45 127) (end 53.92 127) (width 0.5) (layer F.Cu) (net 29))
   (segment (start 53.92 127) (end 54.42 126.5) (width 0.25) (layer F.Cu) (net 29))
   (segment (start 74.25 128.55) (end 74.25 127.85) (width 0.25) (layer F.Cu) (net 30))
@@
       (pts
         (xy 55.7 124.7) (xy 53.1 124.7) (xy 51.5 126.3) (xy 49.2 126.3) (xy 47.3 128.2)
-        (xy 44.6 128.2) (xy 44.6 124.6) (xy 47.8 124.6) (xy 47.8 123.3) (xy 48.5 123.3)
+        (xy 44.6 128.2) (xy 44.6 124.6) (xy 47.8 124.6) (xy 48.5 124.6) (xy 48.5 123.3)
         (xy 48.5 119.1) (xy 56.9 119.1) (xy 56.9 123.5) (xy 56.8 123.5)
       )
